File: Talker.kicad_pcb (KiCad board)
At the start: 2 copper layers, 99.9 x 99.9 mm, 65 parts, among them J1 DC_JACK, J2 DE9, J3 Audio Out, J4 TxE, J5 SPKR, J6 32/16, P1 10K, SW1 RESET, U1 CTS256A-AL2, U10 2732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

Commit message: Modified the circuit to add a negative supply for the op-amp. It made a world of difference!
Parts:
- added C30: 10uF, modules:CP_Radial_D5.0mm_P2.00mm, F.Cu at (128.3, 84.5)
- added C31: 2.2uF, modules:C_Disc_D3_P2.5, F.Cu at (127.0, 81.3)
- added U9: ICL7660, modules:DIP-8_W7.62mm_LongPads, F.Cu at (115.6, 78.7)
- moved C10 46.7 mm to (110.5, 81.3), turned to 270 degrees
- moved C26 24.5 mm to (133.3, 107.3), turned to 90 degrees
Connections:
- U5 pad 11: GND -> V-
- U6 pad 1: Net-(C10-Pad1) -> Net-(U6-Pad1)
- U6 pad 8: Net-(C10-Pad2) -> Net-(U6-Pad8)
Routing:
- net V-: track 0.00 -> 54.2 mm, vias 0 -> 1
- net Net-(C13-Pad2): track 37.0 -> 30.6 mm
- net +5V: track 391.1 -> 395.8 mm, vias 6 -> 4
- net Net-(U4-Pad24): track 13.0 -> 14.5 mm
- net Net-(C10-Pad1): track 6.50 -> 5.08 mm
Other:
- board text added: "GI CTS256-AL2/SPO256-AL2 Text to speech board Vers 1.1 Mar 27 2023"
- board text added: "GI CTS256-AL2/SPO256-AL2 Text to speech board Vers 2.0 Mar 20 2023"
- board text removed: "GI CTS256-AL2/SPO256-AL2 text to speech board Vers 1.0 Feb 4 2023"
